File: CMOS Flash Memory.sch (KiCad schematic (older format))
At the start: 2 parts, among them U5 28F010, U7 28F010

Commit message: bruh
Parts:
- U5, U7: symbol 28F010:28F010 -> proj5-rescue:28F010-28F010
Changed lines of the file:
@@
 $Descr A4 11693 8268
 encoding utf-8
-Sheet 2 5
+Sheet 2 4
 Title ""
 Date ""
@@
 $EndDescr
 $Comp
-L 28F010:28F010 U5
+L proj5-rescue:28F010-28F010 U5
 U 1 1 5E9B9D1A
 P 2600 2950
@@
 	4800 3950 5400 3950
 $Comp
-L 28F010:28F010 U7
+L proj5-rescue:28F010-28F010 U7
 U 1 1 5E9C1E63
 P 7150 2800
