File: CMOS Flash Memory.sch (KiCad schematic (older format))
At the start: 2 parts, among them U5 28F010, U7 28F010

Commit message: sfds
Other:
- moved on the sheet: U7
Changed lines of the file:
@@
 L 28F010:28F010 U7
 U 1 1 5E9C1E63
-P 7150 2800
-F 0 "U7" H 8250 3187 60  0000 C CNN
-F 1 "28F010" H 8250 3081 60  0000 C CNN
-F 2 "28F010" H 8250 3040 60  0001 C CNN
-F 3 "" H 7150 2800 60  0000 C CNN
-	1    7150 2800
+P 6500 2900
+F 0 "U7" H 7600 3287 60  0000 C CNN
+F 1 "28F010" H 7600 3181 60  0000 C CNN
+F 2 "28F010" H 7600 3140 60  0001 C CNN
+F 3 "" H 6500 2900 60  0000 C CNN
+	1    6500 2900
 	1    0    0    -1
 $EndComp
 Wire Bus Line
-	7150 4000 7150 4200
+	6500 4100 6500 4300
 Wire Bus Line
-	7150 4200 6850 4200
+	6500 4300 6200 4300
 Wire Bus Line
-	6850 4200 6850 4600
+	6200 4300 6200 4700
 Wire Bus Line
-	6850 4600 9350 4600
+	6200 4700 8700 4700
 Wire Bus Line
-	9350 4600 9350 3900
+	8700 4700 8700 4000
 Wire Bus Line
-	9350 3900 9600 3900
-Text GLabel 9600 3900 2    50   Input ~ 0
+	8700 4000 8950 4000
+Text GLabel 8950 4000 2    50   Input ~ 0
 DB[0:7]
 Wire Bus Line
-	9350 3700 9500 3700
+	8700 3800 8850 3800
 Wire Bus Line
-	9500 3700 9500 3500
+	8850 3800 8850 3600
 Wire Bus Line
-	9500 3500 9350 3500
+	8850 3600 8700 3600
 Wire Bus Line
-	9350 3500 9350 3100
+	8700 3600 8700 3200
 Wire Bus Line
-	9350 3100 9550 3100
-Text GLabel 9550 3100 2    50   Input ~ 0
+	8700 3200 8900 3200
+Text GLabel 8900 3200 2    50   Input ~ 0
 AB[0:16]
 Wire Bus Line
-	7150 3900 7150 2900
+	6500 4000 6500 3000
 Wire Bus Line
-	7150 2900 6800 2900
-Text GLabel 6800 2900 0    50   Input ~ 0
+	6500 3000 6150 3000
+Text GLabel 6150 3000 0    50   Input ~ 0
 AB[0:16]
 Wire Wire Line
-	9350 3600 9950 3600
+	8700 3700 9300 3700
 Wire Wire Line
-	9350 2900 9850 2900
+	8700 3000 9200 3000
 $Comp
 L power:VCC #PWR?
 U 1 1 5E9C1E7B
-P 9750 2750
-F 0 "#PWR?" H 9750 2600 50  0001 C CNN
-F 1 "VCC" H 9767 2923 50  0000 C CNN
-F 2 "" H 9750 2750 50  0001 C CNN
-F 3 "" H 9750 2750 50  0001 C CNN
-	1    9750 2750
+P 9100 2850
+F 0 "#PWR?" H 9100 2700 50  0001 C CNN
+F 1 "VCC" H 9117 3023 50  0000 C CNN
+F 2 "" H 9100 2850 50  0001 C CNN
+F 3 "" H 9100 2850 50  0001 C CNN
+	1    9100 2850
 	1    0    0    -1
 $EndComp
 Wire Wire Line
-	9750 2750 9750 2800
+	9100 2850 9100 2900
 Wire Wire Line
-	9350 2800 9750 2800
-Text Label 9850 2900 0    50   ~ 0
+	8700 2900 9100 2900
+Text Label 9200 3000 0    50   ~ 0
 HighWR
-Text Label 9950 3600 0    50   ~ 0
+Text Label 9300 3700 0    50   ~ 0
 RD
-Text Label 9950 3750 0    50   ~ 0
+Text Label 9300 3850 0    50   ~ 0
 FlashENABLE
 Wire Wire Line
-	9950 3750 9950 3800
+	9300 3850 9300 3900
 Wire Wire Line
-	9350 3800 9950 3800
+	8700 3900 9300 3900
 $EndSCHEMATC

Commit message: update
Parts:
- removed U5, U7: 28F010, 28F010, symbol 28F010:28F010
- added U? (x2): 28F010, 28F010, symbol 28F010:28F010
- added U?: PAL16L8, symbol Logic_Programmable:PAL16L8
- added U? (x2): 74LS32, symbol 74xx:74LS32
- added U? (x2): 74LS04, symbol 74xx:74LS04
Connections:
- new net: U?.1, U?.3, U?.3
- new net AB0: U?.1
- new net AB1: U?.12 (A0), U?.12 (A0)
- new net AB10: U?.26 (A9)
- new net AB11: U?.23 (A10)
- new net AB12: U?.25 (A11)
- new net AB13: U?.4 (A12), U?.4 (A12)
- new net AB14: U?.28 (A13)
- new net AB15: U?.29 (A14)
- new net AB16: U?.3 (A15), U?.3 (A15)
- new net AB17: U?.2 (A16), U?.2 (A16)
- new net AB18: U?.1 (I1)
- new net AB19: U?.2 (I2)
- new net AB2: U?.11 (A1), U?.11 (A1)
- new net AB3: U?.10 (A2), U?.10 (A2)
- new net AB4: U?.9 (A3), U?.9 (A3)
- new net AB5: U?.8 (A4), U?.8 (A4)
- new net AB6: U?.7 (A5), U?.7 (A5)
- new net AB7: U?.6 (A6), U?.6 (A6)
- new net AB8: U?.5 (A7), U?.5 (A7)
- new net AB9: U?.27 (A8)
- new net BHE: U?.2
- new net FFFFFh: U?.1, U?.19 (IO1), U?.2, U?.22 (CE), U?.22 (CE)
- new net WE: U?.2, U?.31 (WE)
- new net WR: U?.1, U?.2

Commit message: sram v1
Changed lines of the file:
@@
 $Descr A4 11693 8268
 encoding utf-8
-Sheet 2 7
+Sheet 2 8
 Title ""
 Date ""
@@
 Text HLabel 7650 2800 2    50   Input ~ 0
 ADDRESS_BUS
-Wire Bus Line
-	7400 2800 7400 4500
-Wire Bus Line
-	6800 4400 6800 5350
-Wire Bus Line
-	6700 2800 6700 4300
-Wire Bus Line
-	3450 3500 3450 4500
 Wire Wire Line
 	6550 4600 6150 4600
@@
 	1    0    0    1
 $EndComp
+Wire Bus Line
+	6800 4400 6800 5350
+Wire Bus Line
+	6700 2800 6700 4300
+Wire Bus Line
+	7400 2800 7400 4500
+Wire Bus Line
+	3450 3500 3450 4500
+Text HLabel 4850 2600 0    50   Input ~ 0
+DATA_BUS
+Text HLabel 5750 2600 0    50   Input ~ 0
+CONTROL_BUS
 $EndSCHEMATC

Commit message: thur-23
Parts:
- gave numbers to parts that had none: 7
Connections:
- net AB10: now also U6.26 (A9)
- net AB11: now also U6.23 (A10)
- net AB12: now also U6.25 (A11)
- net AB14: now also U6.28 (A13)
- net AB15: now also U6.29 (A14)
- net AB9: now also U6.27 (A8)
- net WE: now also U1.3, U2.3, U4.1, U6.31 (WE)
- net GND: now reaches U3.1 (VPP)
- net GND: now also U3.16 (VSS), U5.10 (GND), U6.1 (VPP), U6.16 (VSS)
- net DB0: now reaches U3.13 (DQ0)
- net DB0: now also U6.13 (DQ0)
- net DB1: now reaches U3.14 (DQ1)
- net DB1: now also U6.14 (DQ1)
- net DB2: now reaches U3.15 (DQ2)
- net DB2: now also U6.15 (DQ2)
- net DB3: now reaches U3.17 (DQ3)
- net DB3: now also U6.17 (DQ3)
- net DB4: now reaches U3.18 (DQ4)
- net DB4: now also U6.18 (DQ4)
- net DB5: now reaches U3.19 (DQ5)
- net DB5: now also U6.19 (DQ5)
- net DB6: now reaches U3.20 (DQ6)
- net DB6: now also U6.20 (DQ6)
- net DB7: now reaches U3.21 (DQ7)
- net DB7: now also U6.21 (DQ7)
- net RD: now reaches U3.24 (OE)
- net RD: now also U6.24 (OE)
- net VCC: now reaches U3.32 (VCC)
- net VCC: now also U5.20 (VCC), U6.32 (VCC)
- net AB16 renamed A16
- net AB17 renamed A17
- net AB18 renamed A18
- net AB19 renamed A19
- net BHE renamed -BHE
- no-connect marks 0 -> 17
Other:
- moved on the sheet: U4A, U7A
