File: proj5.sch (KiCad schematic (older format))
At the start: 0 parts

Commit message: bruh
Changed lines of the file:
@@
 $Descr A4 11693 8268
 encoding utf-8
-Sheet 1 5
+Sheet 1 4
 Title ""
 Date ""
@@
 $EndSheet
 $Sheet
-S 2600 3300 1950 650
-U 5E9BB470
-F0 "Sheet5E9BB46F" 50
-F1 "shit might be done.sch" 50
-$EndSheet
-$Sheet
-S 7400 3350 800  350
-U 5E9BB6A3
-F0 "Sheet5E9BB6A2" 50
-F1 "asdfasdf.sch" 50
+S 4750 2950 850  250
+U 5E9CD8B5
+F0 "SRAM" 50
+F1 "SRAM.sch" 50
 $EndSheet
 $EndSCHEMATC
