File: proj5.sch (KiCad schematic (older format))
At the start: 0 parts

Commit message: sfds
Changed lines of the file:
@@
 S 1900 1550 850  350
 U 5E9B9C0C
-F0 "Sheet5E9B9C0B" 50
+F0 "CMOS" 50
 F1 "CMOS Flash Memory.sch" 50
 $EndSheet
 $Sheet
-S 8350 2050 1500 500
+S 4650 1350 1500 500
 U 5E9BAC16
 F0 "8086" 50

Commit message: 16550 v1
Changed lines of the file:
@@
 $Descr A4 11693 8268
 encoding utf-8
-Sheet 1 5
+Sheet 1 7
 Title ""
 Date ""
@@
 $EndSheet
 $Sheet
-S 2600 3300 1950 650
-U 5E9BB470
-F0 "Sheet5E9BB46F" 50
-F1 "shit might be done.sch" 50
-$EndSheet
-$Sheet
 S 7400 3350 800  350
 U 5E9BB6A3
@@
 F1 "asdfasdf.sch" 50
 $EndSheet
+$Sheet
+S 1900 2400 1550 450
+U 5EFDD26F
+F0 "Clock Generator" 50
+F1 "ClockGen.sch" 50
+$EndSheet
+$Sheet
+S 5000 2550 1150 450
+U 5EFF525E
+F0 "Headers" 50
+F1 "Headers.sch" 50
+$EndSheet
+$Sheet
+S 2450 3350 1150 700
+U 5F01E68D
+F0 "16550 UART" 50
+F1 "16550.sch" 50
+$EndSheet
 $EndSCHEMATC

Commit message: update
Changed lines of the file:
@@
 $EndDescr
 $Sheet
-S 1900 1550 850  350
+S 4950 3450 850  350
 U 5E9B9C0C
 F0 "CMOS" 50
@@
 F0 "8086" 50
 F1 "8086.sch" 50
+F2 "ADDRESS_BUS" O L 4650 1600 50
+F3 "DATA_BUS" I L 4650 1700 50
+F4 "CONTROL_BUS" O L 4650 1500 50
 $EndSheet
 $Sheet
-S 7400 3350 800  350
-U 5E9BB6A3
-F0 "Sheet5E9BB6A2" 50
-F1 "asdfasdf.sch" 50
-$EndSheet
-$Sheet
-S 1900 2400 1550 450
+S 6750 1350 1550 450
 U 5EFDD26F
 F0 "Clock Generator" 50
@@
 $EndSheet
 $Sheet
-S 2450 3350 1150 700
+S 2900 1200 1150 700
 U 5F01E68D
 F0 "16550 UART" 50
 F1 "16550.sch" 50
 $EndSheet
+$Sheet
+S 3200 2650 1150 400
+U 5EB28DAD
+F0 "7 Segment Displays" 50
+F1 "7SegmentDisplays.sch" 50
+$EndSheet
 $EndSCHEMATC

Commit message: sram v1
Connections:
- wire segments 0 -> 37
Changed lines of the file:
@@
 $Descr A4 11693 8268
 encoding utf-8
-Sheet 1 7
+Sheet 1 8
 Title ""
 Date ""
@@
 $EndDescr
 $Sheet
-S 4950 3450 850  350
+S 7950 3750 850  550
 U 5E9B9C0C
 F0 "CMOS" 50
 F1 "CMOS Flash Memory.sch" 50
+F2 "ADDRESS_BUS" I L 7950 4000 50
+F3 "DATA_BUS" I L 7950 4150 50
+F4 "CONTROL_BUS" I L 7950 3850 50
 $EndSheet
 $Sheet
-S 4650 1350 1500 500
-U 5E9BAC16
-F0 "8086" 50
-F1 "8086.sch" 50
-F2 "ADDRESS_BUS" O L 4650 1600 50
-F3 "DATA_BUS" I L 4650 1700 50
-F4 "CONTROL_BUS" O L 4650 1500 50
-$EndSheet
-$Sheet
-S 6750 1350 1550 450
-U 5EFDD26F
-F0 "Clock Generator" 50
-F1 "ClockGen.sch" 50
-$EndSheet
-$Sheet
-S 5000 2550 1150 450
+S 5200 2800 850  500
 U 5EFF525E
 F0 "Headers" 50
 F1 "Headers.sch" 50
+F2 "ADDRESS_BUS" I L 5200 3050 50
+F3 "DATA_BUS" I L 5200 3200 50
+F4 "CONTROL_BUS" I L 5200 2900 50
 $EndSheet
 $Sheet
-S 2900 1200 1150 700
+S 1850 1600 1150 700
 U 5F01E68D
 F0 "16550 UART" 50
 F1 "16550.sch" 50
+F2 "ADDRESS_BUS" I L 1850 2100 50
+F3 "PCLK" I L 1850 1950 50
 $EndSheet
 $Sheet
-S 3200 2650 1150 400
+S 5350 5400 1150 400
 U 5EB28DAD
 F0 "7 Segment Displays" 50
 F1 "7SegmentDisplays.sch" 50
 $EndSheet
+$Sheet
+S 7850 2150 900  550
+U 5EA11F57
+F0 "SRAM" 50
+F1 "SRAM.sch" 50
+F2 "ADDRESS_BUS" I L 7850 2400 50
+F3 "DATA_BUS" O L 7850 2550 50
+F4 "CONTROL_BUS" I L 7850 2250 50
+$EndSheet
+Wire Wire Line
+	4800 3850 4800 2900
+Wire Wire Line
+	4800 2900 5200 2900
+Connection ~ 4800 3850
+Wire Wire Line
+	4800 3850 7250 3850
+Wire Wire Line
+	4900 4000 4900 3050
+Wire Wire Line
+	4900 3050 5200 3050
+Connection ~ 4900 4000
+Wire Wire Line
+	4900 4000 7950 4000
+Wire Wire Line
+	5200 3200 5000 3200
+Wire Wire Line
+	5000 3200 5000 4150
+Connection ~ 5000 4150
+Wire Wire Line
+	5000 4150 7550 4150
+Wire Wire Line
+	7250 3850 7250 2250
+Wire Wire Line
+	7250 2250 7850 2250
+Connection ~ 7250 3850
+Wire Wire Line
+	7250 3850 7950 3850
+Wire Wire Line
+	7400 3950 7400 2400
+Wire Wire Line
+	7400 2400 7850 2400
+Wire Wire Line
+	7550 4150 7550 2550
+Wire Wire Line
+	7550 2550 7850 2550
+Connection ~ 7550 4150
+Wire Wire Line
+	7550 4150 7950 4150
+Wire Wire Line
+	2950 3850 4800 3850
+Wire Wire Line
+	2950 4150 5000 4150
+Wire Wire Line
+	2950 4000 3600 4000
+$Sheet
+S 1500 3450 1450 1650
+U 5E9BAC16
+F0 "8086" 50
+F1 "8086.sch" 50
+F2 "ADDRESS_BUS" O R 2950 4000 50
+F3 "DATA_BUS" O R 2950 4150 50
+F4 "CONTROL_BUS" O R 2950 3850 50
+F5 "CLK" I L 1500 3850 50
+F6 "READY" I L 1500 4000 50
+F7 "RESET" I L 1500 4150 50
+$EndSheet
+Wire Wire Line
+	3600 4000 3600 3200
+Wire Wire Line
+	3600 3200 900  3200
+Wire Wire Line
+	900  3200 900  2100
+Wire Wire Line
+	900  2100 1850 2100
+Connection ~ 3600 4000
+Wire Wire Line
+	3600 4000 4900 4000
+Wire Wire Line
+	750  1950 1850 1950
+Wire Wire Line
+	1300 5850 1300 4150
+Wire Wire Line
+	1300 4150 1500 4150
+Wire Wire Line
+	1150 6000 1150 4000
+Wire Wire Line
+	1150 4000 1500 4000
+Wire Wire Line
+	950  3850 1500 3850
+Wire Wire Line
+	950  3850 950  6150
+Wire Wire Line
+	1500 5850 1300 5850
+Wire Wire Line
+	1500 6000 1150 6000
+Wire Wire Line
+	950  6150 1500 6150
+Wire Wire Line
+	750  6300 750  1950
+$Sheet
+S 1500 5650 1400 900
+U 5EFDD26F
+F0 "Clock Generator" 50
+F1 "ClockGen.sch" 50
+F2 "CLK" I L 1500 6150 50
+F3 "READY" I L 1500 6000 50
+F4 "RESET" I L 1500 5850 50
+F5 "PCLK" I L 1500 6300 50
+$EndSheet
+Wire Wire Line
+	750  6300 1500 6300
 $EndSCHEMATC

Commit message: thur-23
Connections:
- wire segments 37 -> 30
Changed lines of the file:
@@
 $Descr A4 11693 8268
 encoding utf-8
-Sheet 1 8
+Sheet 1 6
 Title ""
 Date ""
@@
 $EndSheet
 $Sheet
-S 1850 1600 1150 700
-U 5F01E68D
-F0 "16550 UART" 50
-F1 "16550.sch" 50
-F2 "ADDRESS_BUS" I L 1850 2100 50
-F3 "PCLK" I L 1850 1950 50
-$EndSheet
-$Sheet
-S 5350 5400 1150 400
-U 5EB28DAD
-F0 "7 Segment Displays" 50
-F1 "7SegmentDisplays.sch" 50
-$EndSheet
-$Sheet
 S 7850 2150 900  550
 U 5EA11F57
@@
 Connection ~ 4900 4000
 Wire Wire Line
-	4900 4000 7950 4000
+	4900 4000 7400 4000
 Wire Wire Line
 	5200 3200 5000 3200
@@
 	7250 3850 7950 3850
 Wire Wire Line
-	7400 3950 7400 2400
-Wire Wire Line
 	7400 2400 7850 2400
 Wire Wire Line
@@
 Wire Wire Line
 	2950 4150 5000 4150
-Wire Wire Line
-	2950 4000 3600 4000
 $Sheet
 S 1500 3450 1450 1650
@@
 F7 "RESET" I L 1500 4150 50
 $EndSheet
-Wire Wire Line
-	3600 4000 3600 3200
-Wire Wire Line
-	3600 3200 900  3200
-Wire Wire Line
-	900  3200 900  2100
-Wire Wire Line
-	900  2100 1850 2100
-Connection ~ 3600 4000
-Wire Wire Line
-	3600 4000 4900 4000
-Wire Wire Line
-	750  1950 1850 1950
 Wire Wire Line
 	1300 5850 1300 4150
@@
 Wire Wire Line
 	950  6150 1500 6150
-Wire Wire Line
-	750  6300 750  1950
 $Sheet
 S 1500 5650 1400 900
@@
 $EndSheet
 Wire Wire Line
-	750  6300 1500 6300
+	7400 2400 7400 4000
+Connection ~ 7400 4000
+Wire Wire Line
+	7400 4000 7950 4000
+Wire Wire Line
+	2950 4000 4900 4000
 $EndSCHEMATC
