File: Headers.sch (KiCad schematic (older format))
At the start: 0 parts

Commit message: 8086 v2
Parts:
- added J?: Conn_02x30_Top_Bottom, symbol Connector_Generic:Conn_02x30_Top_Bottom
Changed lines of the file:
@@
 $Descr A4 11693 8268
 encoding utf-8
-Sheet 7 7
+Sheet 6 7
 Title ""
 Date ""
@@
 Comment4 ""
 $EndDescr
+$Comp
+L Connector_Generic:Conn_02x30_Top_Bottom J?
+U 1 1 5EA32CD9
+P 5350 4150
+F 0 "J?" H 5400 5767 50  0000 C CNN
+F 1 "Conn_02x30_Top_Bottom" H 5400 5676 50  0000 C CNN
+F 2 "" H 5350 4150 50  0001 C CNN
+F 3 "~" H 5350 4150 50  0001 C CNN
+	1    5350 4150
+	1    0    0    -1
+$EndComp
 $EndSCHEMATC
