File: 16550.sch (KiCad schematic (older format))
At the start: 4 parts

Commit message: update
Connections:
- net labels added: ADDRESS_BUS
Changed lines of the file:
@@
 $Descr A4 11693 8268
 encoding utf-8
-Sheet 7 7
+Sheet 6 7
 Title ""
 Date ""
@@
 	1    0    0    -1
 $EndComp
-Text GLabel 2150 3400 0    50   Input ~ 0
-PCLK(8284)
 Text GLabel 4500 4400 2    50   Input ~ 0
 RCLK
@@
 BAUDOUT
 $Comp
-L power:GND #PWR?
+L power:GND #PWR0114
 U 1 1 5F06B893
 P 10050 4400
-F 0 "#PWR?" H 10050 4150 50  0001 C CNN
+F 0 "#PWR0114" H 10050 4150 50  0001 C CNN
 F 1 "GND" H 10055 4227 50  0000 C CNN
 F 2 "" H 10050 4400 50  0001 C CNN
@@
 $EndComp
 $Comp
-L power:GND #PWR?
+L power:GND #PWR0115
 U 1 1 5F05F720
 P 6000 2700
-F 0 "#PWR?" H 6000 2450 50  0001 C CNN
+F 0 "#PWR0115" H 6000 2450 50  0001 C CNN
 F 1 "GND" H 6005 2527 50  0000 C CNN
 F 2 "" H 6000 2700 50  0001 C CNN
@@
 Wire Wire Line
 	4300 4400 4500 4400
-Wire Wire Line
-	2300 3400 2150 3400
 Wire Bus Line
 	2150 1550 1750 1550
@@
 	1950 4350 1950 4850
 $Comp
-L power:GND #PWR?
+L power:GND #PWR0116
 U 1 1 5F08B71A
 P 1950 4850
-F 0 "#PWR?" H 1950 4600 50  0001 C CNN
+F 0 "#PWR0116" H 1950 4600 50  0001 C CNN
 F 1 "GND" H 1955 4677 50  0000 C CNN
 F 2 "" H 1950 4850 50  0001 C CNN
@@
 	1    0    0    -1
 $EndComp
+Text HLabel 1750 1550 0    50   Input ~ 0
+ADDRESS_BUS
+Text GLabel 2150 3400 0    50   Input ~ 0
+PCLK(8284)
 Wire Bus Line
 	2150 2500 2150 3050
 Wire Bus Line
 	2150 1550 2150 2350
+Wire Wire Line
+	2300 3400 2150 3400
 $EndSCHEMATC

Commit message: sram v1
Connections:
- net labels added: PCLK
- net labels removed: PCLK(8284)
Changed lines of the file:
@@
 $Descr A4 11693 8268
 encoding utf-8
-Sheet 6 7
+Sheet 4 8
 Title ""
 Date ""
@@
 Text HLabel 1750 1550 0    50   Input ~ 0
 ADDRESS_BUS
-Text GLabel 2150 3400 0    50   Input ~ 0
-PCLK(8284)
+Text GLabel 2200 3350 0    50   Input ~ 0
+PCLK
+Wire Wire Line
+	1600 3350 2450 3350
+Text HLabel 1600 3350 0    50   Input ~ 0
+PCLK
 Wire Bus Line
 	2150 2500 2150 3050
 Wire Bus Line
 	2150 1550 2150 2350
-Wire Wire Line
-	2300 3400 2150 3400
 $EndSCHEMATC

Commit message: thur-23
Parts:
- gave numbers to parts that had none: 4
Changed lines of the file:
@@
 $EndDescr
 $Comp
-L Logic_Programmable:PAL16L8 U?
+L Logic_Programmable:PAL16L8 U9
 U 1 1 5F027763
 P 5300 6650
-F 0 "U?" H 5300 7531 50  0000 C CNN
+F 0 "U9" H 5300 7531 50  0000 C CNN
 F 1 "PAL16L8" H 5300 7440 50  0000 C CNN
 F 2 "" H 5300 6650 50  0001 C CNN
@@
 $EndComp
 $Comp
-L max235cpg:max235cpg U?
+L max235cpg:max235cpg U10
 U 1 1 5F023538
 P 7350 3050
-F 0 "U?" H 8650 3437 60  0000 C CNN
+F 0 "U10" H 8650 3437 60  0000 C CNN
 F 1 "max235cpg" H 8650 3331 60  0000 C CNN
 F 2 "max235cpg" H 8650 3290 60  0001 C CNN
@@
 BAUDOUT
 $Comp
-L power:GND #PWR0114
+L power:GND #PWR011
 U 1 1 5F06B893
 P 10050 4400
-F 0 "#PWR0114" H 10050 4150 50  0001 C CNN
+F 0 "#PWR011" H 10050 4150 50  0001 C CNN
 F 1 "GND" H 10055 4227 50  0000 C CNN
 F 2 "" H 10050 4400 50  0001 C CNN
@@
 $EndComp
 $Comp
-L DSUB-9:DSUB-9 J?
+L DSUB-9:DSUB-9 J2
 U 1 1 5F01F87E
 P 6050 1750
-F 0 "J?" H 6878 1403 60  0000 L CNN
+F 0 "J2" H 6878 1403 60  0000 L CNN
 F 1 "DSUB-9" H 6878 1297 60  0000 L CNN
 F 2 "DSUB-9" H 6650 1390 60  0001 C CNN
@@
 $EndComp
 $Comp
-L power:GND #PWR0115
+L power:GND #PWR010
 U 1 1 5F05F720
 P 6000 2700
-F 0 "#PWR0115" H 6000 2450 50  0001 C CNN
+F 0 "#PWR010" H 6000 2450 50  0001 C CNN
 F 1 "GND" H 6005 2527 50  0000 C CNN
 F 2 "" H 6000 2700 50  0001 C CNN
@@
 	4500 2050 4500 1750
 $Comp
-L Interface_UART:16550 U?
+L Interface_UART:16550 U8
 U 1 1 5F01E86F
 P 3450 3150
-F 0 "U?" H 3450 5031 50  0000 C CNN
+F 0 "U8" H 3450 5031 50  0000 C CNN
 F 1 "16550" H 3450 4940 50  0000 C CNN
 F 2 "Package_DIP:DIP-40_W15.24mm" H 3450 3150 50  0001 C CIN
@@
 	1950 4350 1950 4850
 $Comp
-L power:GND #PWR0116
+L power:GND #PWR09
 U 1 1 5F08B71A
 P 1950 4850
-F 0 "#PWR0116" H 1950 4600 50  0001 C CNN
+F 0 "#PWR09" H 1950 4600 50  0001 C CNN
 F 1 "GND" H 1955 4677 50  0000 C CNN
 F 2 "" H 1950 4850 50  0001 C CNN
