File: ClockGen.sch (KiCad schematic (older format))
At the start: 3 parts

Commit message: update
Parts:
- added 10uF: CAP, symbol pspice:CAP
- added D1: DIODE, symbol pspice:DIODE
- added SW?: SW_DPST_x2, symbol Switch:SW_DPST_x2
- gave numbers to parts that had none: 3
Connections:
- net GND: now also U1.9 (GND), 10uF.2, SW?.2 (B)
- net READY: no longer U1.10 (RESET)
- net at U1.11 (~RES~): now also R1.2, 10uF.1, D1.1 (K), SW?.1 (A)
- net VCC: now reaches U1.4 (RDY1)
- net VCC: now also R1.1, D1.2 (A)
- net PCLK renamed PCLK(8284)
- new net RESET: U1.10 (RESET)
- no-connect marks 0 -> 5
Other:
- moved on the sheet: R1, U1
Changed lines of the file:
@@
 $Descr A4 11693 8268
 encoding utf-8
-Sheet 5 7
+Sheet 4 7
 Title ""
 Date ""
@@
 Comment4 ""
 $EndDescr
-$Comp
-L Timer:8284 U?
-U 1 1 5EFDD54D
-P 5550 3800
-F 0 "U?" H 5550 4881 50  0000 C CNN
-F 1 "8284" H 5550 4790 50  0000 C CNN
-F 2 "Package_DIP:DIP-18_W7.62mm" H 5550 3800 50  0001 C CIN
-F 3 "http://www.cpu-galaxy.at/cpu/ram%20rom%20eprom/other_intel_chips/other_intel-Dateien/D8284A_Datasheet.pdf" H 5550 3800 50  0001 C CNN
-	1    5550 3800
-	1    0    0    -1
-$EndComp
-Text GLabel 6600 3200 0    50   Input ~ 0
+Text GLabel 6450 3200 2    50   Output ~ 0
 CLK
 Wire Wire Line
-	6250 3200 6600 3200
-Wire Wire Line
-	6250 3800 6600 3800
-Text GLabel 6600 3800 0    50   Input ~ 0
-PCLK
-Wire Wire Line
-	6250 3400 6600 3400
-Text GLabel 6600 3400 0    50   Input ~ 0
-READY
-Wire Wire Line
-	6250 3600 6600 3600
-Text GLabel 6600 3600 0    50   Input ~ 0
-READY
-Wire Wire Line
-	6250 4200 6500 4200
+	6200 3200 6450 3200
+Wire Wire Line
+	6200 3800 6600 3800
+Wire Wire Line
+	6200 3400 6600 3400
+Wire Wire Line
+	6200 3600 6600 3600
+Text GLabel 6600 3600 2    50   Input ~ 0
+RESET
+Wire Wire Line
+	6200 4200 6500 4200
 Wire Wire Line
 	6500 4200 6500 4150
 Wire Wire Line
-	6250 4400 6500 4400
+	6200 4400 6500 4400
 Wire Wire Line
 	6500 4400 6500 4450
@@
 	6500 4150 6600 4150
 $Comp
-L Device:Crystal Y?
+L Device:Crystal Y1
 U 1 1 5F009BAD
 P 6600 4300
-F 0 "Y?" V 6554 4431 50  0000 L CNN
+F 0 "Y1" V 6554 4431 50  0000 L CNN
 F 1 "Crystal" V 6645 4431 50  0000 L CNN
 F 2 "" H 6600 4300 50  0001 C CNN
@@
 	6500 4450 6600 4450
 $Comp
+L power:GND #PWR0113
+U 1 1 5F0140EC
+P 4650 4600
+F 0 "#PWR0113" H 4650 4350 50  0001 C CNN
+F 1 "GND" H 4655 4427 50  0000 C CNN
+F 2 "" H 4650 4600 50  0001 C CNN
+F 3 "" H 4650 4600 50  0001 C CNN
+	1    4650 4600
+	1    0    0    -1
+$EndComp
+Wire Wire Line
+	4650 4000 4650 4200
+Wire Wire Line
+	4650 4000 4800 4000
+Wire Wire Line
+	4650 4200 4800 4200
+Connection ~ 4650 4200
+$Comp
+L Device:R_Small_US R1
+U 1 1 5F0181BE
+P 4500 5300
+F 0 "R1" V 4295 5300 50  0000 C CNN
+F 1 "10k" V 4386 5300 50  0000 C CNN
+F 2 "" H 4500 5300 50  0001 C CNN
+F 3 "~" H 4500 5300 50  0001 C CNN
+	1    4500 5300
+	0    1    1    0
+$EndComp
+$Comp
+L power:GND #PWR02
+U 1 1 5EABAEA9
+P 5500 4700
+F 0 "#PWR02" H 5500 4450 50  0001 C CNN
+F 1 "GND" H 5505 4527 50  0000 C CNN
+F 2 "" H 5500 4700 50  0001 C CNN
+F 3 "" H 5500 4700 50  0001 C CNN
+	1    5500 4700
+	1    0    0    -1
+$EndComp
+NoConn ~ 6200 3900
+Wire Wire Line
+	4800 3400 4550 3400
+Wire Wire Line
+	4550 3400 4550 2700
+$Comp
+L power:VCC #PWR01
+U 1 1 5EABD349
+P 4550 2700
+F 0 "#PWR01" H 4550 2550 50  0001 C CNN
+F 1 "VCC" H 4567 2873 50  0000 C CNN
+F 2 "" H 4550 2700 50  0001 C CNN
+F 3 "" H 4550 2700 50  0001 C CNN
+	1    4550 2700
+	1    0    0    -1
+$EndComp
+$Comp
+L Timer:8284 U1
+U 1 1 5EFDD54D
+P 5500 3800
+F 0 "U1" H 5500 4150 50  0000 C CNN
+F 1 "8284" H 5500 4000 50  0000 C CNN
+F 2 "Package_DIP:DIP-18_W7.62mm" H 5500 3800 50  0001 C CIN
+F 3 "http://www.cpu-galaxy.at/cpu/ram%20rom%20eprom/other_intel_chips/other_intel-Dateien/D8284A_Datasheet.pdf" H 5500 3800 50  0001 C CNN
+	1    5500 3800
+	1    0    0    -1
+$EndComp
+NoConn ~ 4800 3600
+NoConn ~ 4800 3700
+Wire Wire Line
+	4650 4200 4650 4600
+NoConn ~ 4800 4400
+NoConn ~ 4800 3900
+Wire Wire Line
+	4800 3200 4200 3200
+Wire Wire Line
+	4200 5300 4400 5300
+Wire Wire Line
+	4600 5300 5150 5300
+$Comp
+L pspice:DIODE D1
+U 1 1 5EAC3FA1
+P 4600 5700
+F 0 "D1" H 4600 5965 50  0000 C CNN
+F 1 "DIODE" H 4600 5874 50  0000 C CNN
+F 2 "" H 4600 5700 50  0001 C CNN
+F 3 "~" H 4600 5700 50  0001 C CNN
+	1    4600 5700
+	1    0    0    -1
+$EndComp
+Wire Wire Line
+	4400 5700 4200 5700
+Wire Wire Line
+	4200 5700 4200 5300
+Connection ~ 4200 5300
+Wire Wire Line
+	4800 5700 5150 5700
+Wire Wire Line
+	4200 5700 3850 5700
+Connection ~ 4200 5700
+$Comp
+L pspice:CAP 10uF
+U 1 1 5EACB295
+P 3450 5700
+F 0 "10uF" V 3135 5700 50  0000 C CNN
+F 1 "CAP" V 3226 5700 50  0000 C CNN
+F 2 "" H 3450 5700 50  0001 C CNN
+F 3 "~" H 3450 5700 50  0001 C CNN
+	1    3450 5700
+	0    1    1    0
+$EndComp
+Connection ~ 3850 5700
+Wire Wire Line
+	3850 5700 3700 5700
+Wire Wire Line
+	3850 5700 3850 6100
+Wire Wire Line
+	3850 6100 4200 6100
+Wire Wire Line
+	4600 6100 4850 6100
+Wire Wire Line
+	5150 5300 5350 5300
+Wire Wire Line
+	5350 5300 5350 5250
+Connection ~ 5150 5300
+Wire Wire Line
+	5150 5300 5150 5700
+$Comp
+L power:VCC #PWR?
+U 1 1 5EAD4379
+P 5350 5250
+F 0 "#PWR?" H 5350 5100 50  0001 C CNN
+F 1 "VCC" H 5367 5423 50  0000 C CNN
+F 2 "" H 5350 5250 50  0001 C CNN
+F 3 "" H 5350 5250 50  0001 C CNN
+	1    5350 5250
+	1    0    0    -1
+$EndComp
+$Comp
 L power:GND #PWR?
-U 1 1 5F0140EC
-P 4650 4300
-F 0 "#PWR?" H 4650 4050 50  0001 C CNN
-F 1 "GND" H 4655 4127 50  0000 C CNN
-F 2 "" H 4650 4300 50  0001 C CNN
-F 3 "" H 4650 4300 50  0001 C CNN
-	1    4650 4300
-	1    0    0    -1
-$EndComp
-Wire Wire Line
-	4650 4000 4650 4200
-Wire Wire Line
-	4650 4000 4850 4000
-Wire Wire Line
-	4650 4200 4850 4200
-Connection ~ 4650 4200
-Wire Wire Line
-	4650 4200 4650 4300
-$Comp
-L Device:R_Small_US R?
-U 1 1 5F0181BE
-P 4400 3200
-F 0 "R?" V 4195 3200 50  0000 C CNN
-F 1 "10k" V 4286 3200 50  0000 C CNN
-F 2 "" H 4400 3200 50  0001 C CNN
-F 3 "~" H 4400 3200 50  0001 C CNN
-	1    4400 3200
-	0    1    1    0
-$EndComp
+U 1 1 5EAD4AC7
+P 2850 5700
+F 0 "#PWR?" H 2850 5450 50  0001 C CNN
+F 1 "GND" V 2855 5572 50  0000 R CNN
+F 2 "" H 2850 5700 50  0001 C CNN
+F 3 "" H 2850 5700 50  0001 C CNN
+	1    2850 5700
+	0    1    1    0
+$EndComp
+Wire Wire Line
+	3200 5700 2850 5700
+$Comp
+L power:GND #PWR?
+U 1 1 5EAD7BB6
+P 4850 6200
+F 0 "#PWR?" H 4850 5950 50  0001 C CNN
+F 1 "GND" H 4855 6027 50  0000 C CNN
+F 2 "" H 4850 6200 50  0001 C CNN
+F 3 "" H 4850 6200 50  0001 C CNN
+	1    4850 6200
+	1    0    0    -1
+$EndComp
+Wire Wire Line
+	4850 6100 4850 6200
+Wire Wire Line
+	4200 3200 4200 5300
+Text GLabel 6600 3400 2    50   Input ~ 0
+READY
+$Comp
+L Switch:SW_DPST_x2 SW?
+U 1 1 5EAE475C
+P 4400 6100
+F 0 "SW?" H 4400 6335 50  0000 C CNN
+F 1 "SW_DPST_x2" H 4400 6244 50  0000 C CNN
+F 2 "" H 4400 6100 50  0001 C CNN
+F 3 "~" H 4400 6100 50  0001 C CNN
+	1    4400 6100
+	1    0    0    -1
+$EndComp
+Text GLabel 6600 3800 2    50   Output ~ 0
+PCLK(8284)
 $EndSCHEMATC

Commit message: sram v1
Connections:
- net PCLK(8284) renamed PCLK
Changed lines of the file:
@@
 $Descr A4 11693 8268
 encoding utf-8
-Sheet 4 7
+Sheet 8 8
 Title ""
 Date ""
@@
 Comment4 ""
 $EndDescr
-Text GLabel 6450 3200 2    50   Output ~ 0
+Text GLabel 6450 3200 0    50   Input ~ 0
 CLK
-Wire Wire Line
-	6200 3200 6450 3200
-Wire Wire Line
-	6200 3800 6600 3800
-Wire Wire Line
-	6200 3400 6600 3400
-Wire Wire Line
-	6200 3600 6600 3600
-Text GLabel 6600 3600 2    50   Input ~ 0
+Text GLabel 6550 3600 0    50   Input ~ 0
 RESET
 Wire Wire Line
@@
 Wire Wire Line
 	4200 3200 4200 5300
-Text GLabel 6600 3400 2    50   Input ~ 0
+Text GLabel 6550 3400 0    50   Input ~ 0
 READY
 $Comp
@@
 	1    0    0    -1
 $EndComp
-Text GLabel 6600 3800 2    50   Output ~ 0
-PCLK(8284)
+Text GLabel 6500 3800 0    50   Input ~ 0
+PCLK
+Text HLabel 7200 3200 0    50   Input ~ 0
+CLK
+Wire Wire Line
+	6200 3400 7200 3400
+Wire Wire Line
+	6200 3200 7200 3200
+Text HLabel 7200 3400 0    50   Input ~ 0
+READY
+Wire Wire Line
+	6200 3600 7200 3600
+Text HLabel 7200 3600 0    50   Input ~ 0
+RESET
+Wire Wire Line
+	6200 3800 7200 3800
+Text HLabel 7200 3800 0    50   Input ~ 0
+PCLK
 $EndSCHEMATC

Commit message: thur-23
Parts:
- gave numbers to parts that had none: 1
- renumbered 10uF to 10uF1, D1 to D2, R1 to R2, U1 to U23
Connections:
- net VCC: now also U23.18 (VCC)
Changed lines of the file:
@@
 $Descr A4 11693 8268
 encoding utf-8
-Sheet 8 8
+Sheet 6 6
 Title ""
 Date ""
@@
 	6500 4450 6600 4450
 $Comp
-L power:GND #PWR0113
+L power:GND #PWR043
 U 1 1 5F0140EC
 P 4650 4600
-F 0 "#PWR0113" H 4650 4350 50  0001 C CNN
+F 0 "#PWR043" H 4650 4350 50  0001 C CNN
 F 1 "GND" H 4655 4427 50  0000 C CNN
 F 2 "" H 4650 4600 50  0001 C CNN
@@
 Connection ~ 4650 4200
 $Comp
-L Device:R_Small_US R1
+L Device:R_Small_US R2
 U 1 1 5F0181BE
 P 4500 5300
-F 0 "R1" V 4295 5300 50  0000 C CNN
+F 0 "R2" V 4295 5300 50  0000 C CNN
 F 1 "10k" V 4386 5300 50  0000 C CNN
 F 2 "" H 4500 5300 50  0001 C CNN
@@
 $EndComp
 $Comp
-L power:GND #PWR02
+L power:GND #PWR046
 U 1 1 5EABAEA9
 P 5500 4700
-F 0 "#PWR02" H 5500 4450 50  0001 C CNN
+F 0 "#PWR046" H 5500 4450 50  0001 C CNN
 F 1 "GND" H 5505 4527 50  0000 C CNN
 F 2 "" H 5500 4700 50  0001 C CNN
@@
 	4550 3400 4550 2700
 $Comp
-L power:VCC #PWR01
+L power:VCC #PWR042
 U 1 1 5EABD349
 P 4550 2700
-F 0 "#PWR01" H 4550 2550 50  0001 C CNN
+F 0 "#PWR042" H 4550 2550 50  0001 C CNN
 F 1 "VCC" H 4567 2873 50  0000 C CNN
 F 2 "" H 4550 2700 50  0001 C CNN
@@
 $EndComp
 $Comp
-L Timer:8284 U1
+L Timer:8284 U23
 U 1 1 5EFDD54D
 P 5500 3800
-F 0 "U1" H 5500 4150 50  0000 C CNN
+F 0 "U23" H 5500 4150 50  0000 C CNN
 F 1 "8284" H 5500 4000 50  0000 C CNN
 F 2 "Package_DIP:DIP-18_W7.62mm" H 5500 3800 50  0001 C CIN
@@
 	4600 5300 5150 5300
 $Comp
-L pspice:DIODE D1
+L pspice:DIODE D2
 U 1 1 5EAC3FA1
 P 4600 5700
-F 0 "D1" H 4600 5965 50  0000 C CNN
+F 0 "D2" H 4600 5965 50  0000 C CNN
 F 1 "DIODE" H 4600 5874 50  0000 C CNN
 F 2 "" H 4600 5700 50  0001 C CNN
@@
 Connection ~ 4200 5700
 $Comp
-L pspice:CAP 10uF
+L pspice:CAP 10uF1
 U 1 1 5EACB295
 P 3450 5700
-F 0 "10uF" V 3135 5700 50  0000 C CNN
+F 0 "10uF1" V 3135 5700 50  0000 C CNN
 F 1 "CAP" V 3226 5700 50  0000 C CNN
 F 2 "" H 3450 5700 50  0001 C CNN
@@
 	5150 5300 5150 5700
 $Comp
-L power:VCC #PWR?
+L power:VCC #PWR045
 U 1 1 5EAD4379
 P 5350 5250
-F 0 "#PWR?" H 5350 5100 50  0001 C CNN
+F 0 "#PWR045" H 5350 5100 50  0001 C CNN
 F 1 "VCC" H 5367 5423 50  0000 C CNN
 F 2 "" H 5350 5250 50  0001 C CNN
@@
 $EndComp
 $Comp
-L power:GND #PWR?
+L power:GND #PWR041
 U 1 1 5EAD4AC7
 P 2850 5700
-F 0 "#PWR?" H 2850 5450 50  0001 C CNN
+F 0 "#PWR041" H 2850 5450 50  0001 C CNN
 F 1 "GND" V 2855 5572 50  0000 R CNN
 F 2 "" H 2850 5700 50  0001 C CNN
@@
 	3200 5700 2850 5700
 $Comp
-L power:GND #PWR?
+L power:GND #PWR044
 U 1 1 5EAD7BB6
 P 4850 6200
-F 0 "#PWR?" H 4850 5950 50  0001 C CNN
+F 0 "#PWR044" H 4850 5950 50  0001 C CNN
 F 1 "GND" H 4855 6027 50  0000 C CNN
 F 2 "" H 4850 6200 50  0001 C CNN
@@
 READY
 $Comp
-L Switch:SW_DPST_x2 SW?
+L Switch:SW_DPST_x2 SW2
 U 1 1 5EAE475C
 P 4400 6100
-F 0 "SW?" H 4400 6335 50  0000 C CNN
+F 0 "SW2" H 4400 6335 50  0000 C CNN
 F 1 "SW_DPST_x2" H 4400 6244 50  0000 C CNN
 F 2 "" H 4400 6100 50  0001 C CNN
@@
 Text HLabel 7200 3800 0    50   Input ~ 0
 PCLK
+$Comp
+L power:VCC #PWR0103
+U 1 1 5F628009
+P 5500 2900
+F 0 "#PWR0103" H 5500 2750 50  0001 C CNN
+F 1 "VCC" H 5517 3073 50  0000 C CNN
+F 2 "" H 5500 2900 50  0001 C CNN
+F 3 "" H 5500 2900 50  0001 C CNN
+	1    5500 2900
+	1    0    0    -1
+$EndComp
 $EndSCHEMATC
