File: SRAM.sch (KiCad schematic (older format))
At the start: 8 parts

Commit message: thur-23
Parts:
- gave numbers to parts that had none: 8
Connections:
- net DB10: now also U15.13 (D2)
- net DB11: now also U15.15 (D3)
- net DB12: now also U15.16 (D4)
- net DB13: now also U15.17 (D5)
- net DB14: now also U15.18 (D6)
- net DB15: now also U15.19 (D7)
- net DB8: now also U15.11 (D0)
- net DB9: now also U15.12 (D1)
- net GND: now also U12.22 (~OE~), U13.22 (~OE~), U14.22 (~OE~), U15.22 (~OE~)
- net BHE renamed -BHE
